File: project/contactless-thermometer.brd (EAGLE design)
At the start: 40 x 155 mm, 92 parts, among them J1 OLED, J2 ICSP, J3 BLE, J4 USB-MINIB-5PIN, Q1 MMBT3904, Q2 MMBT3904, Q3 ZXMP6A17GTA, U1 LT1167CS8#PBF, U2 OPA2705UA, U3 OPA705NA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

Commit message: PCB progress
Parts:
- added C22: 0.1uF, SparkFun-Capacitors:0603
- moved R15 60.0 mm to (28.8, 112.7), turned to 0 degrees
- moved C18 38.2 mm to (14.2, 44.1), turned to 270 degrees
- moved J3 36.5 mm to (37.4, 146.0), turned to 270 degrees
- moved S5 33.9 mm to (3.30, 139.6)
- moved TP8 26.9 mm to (37.1, 120.3)
- moved R26 22.0 mm to (32.0, 138.5), turned to 180 degrees
- moved TP7 20.8 mm to (40.6, 105.8)
- moved R25 20.2 mm to (32.0, 135.9), turned to 0 degrees
- moved D2 18.1 mm to (26.4, 50.7), turned to 90 degrees
- moved TP5 17.8 mm to (38.1, 118.5)
- moved C15 15.4 mm to (26.4, 54.0), turned to 0 degrees
- moved R13 15.3 mm to (14.7, 106.6)
- moved C16 14.3 mm to (26.9, 58.9), turned to 90 degrees
- moved U6 11.4 mm to (17.8, 51.2), turned to 90 degrees
- moved R16 11.1 mm to (6.60, 89.2), turned to 0 degrees
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Connections:
- net 3.3V: now also C22.1
- net GND: now also C22.2
- net N$15: now also U5.17; no longer U5.15
- net N$21: now also U5.15; no longer U5.17
Routing:
- net GND: track 0.00 -> 92.9 mm, vias 0 -> 32
- net BLE_TX: track 0.00 -> 70.5 mm
- net VCC: track 0.00 -> 63.1 mm
- net N$28: track 0.00 -> 52.5 mm, vias 0 -> 1
- net N$25: track 0.00 -> 48.4 mm
- net BLE_RX: track 0.00 -> 45.1 mm
- net BUT_L: track 0.00 -> 41.6 mm
- net N$44: track 0.00 -> 37.7 mm
- net BUT_MID: track 0.00 -> 34.6 mm
- net VTH: track 0.00 -> 31.0 mm, vias 0 -> 2
- net RESET: track 0.00 -> 30.2 mm, vias 0 -> 2
- net BUT_R: track 0.00 -> 29.5 mm
- net 5V: track 0.00 -> 27.3 mm
- net LED_G: track 0.00 -> 23.9 mm
- net PWR_OUT: track 0.00 -> 20.4 mm
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- added copper zone on layer 16, net GND
Other:
- board size 40 x 155 mm -> 50 x 150 mm

Commit message: allah
Parts:
- removed TP3: TPTP10R, testpad:TP10R
- moved U3 103.3 mm to (11.4, 132.7), turned to 270 degrees
- moved Q1 102.7 mm to (8.89, 127.4)
- moved R11 99.2 mm to (5.84, 132.3)
- moved R29 99.1 mm to (8.13, 132.3)
- moved R12 98.0 mm to (5.84, 127.3)
- moved TP4 89.4 mm to (7.54, 123.5), turned to 0 degrees
- moved TP6 40.1 mm to (32.3, 70.8)
- moved TP7 25.4 mm to (25.1, 126.0)
- moved TP5 15.8 mm to (22.6, 115.5)
- moved TP8 14.2 mm to (25.1, 127.9)
- moved R3 9.06 mm to (22.3, 124.3), turned to 270 degrees
- moved R24 8.99 mm to (24.3, 74.8), turned to 180 degrees
- moved D4 8.90 mm to (23.6, 15.2), turned to 270 degrees
- moved D3 5.08 mm to (20.8, 15.2), turned to 270 degrees
- moved LS1 2.05 mm to (23.4, 36.0)
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Connections:
- net 2.5V: no longer TP3.TP
Routing:
- net PWR_OUT: track 20.4 -> 158.6 mm, vias 0 -> 2
- net RESET: track 30.2 -> 146.3 mm, vias 2 -> 4
- net PWR_IN: track 18.3 -> 131.3 mm, vias 0 -> 2
- net N$9: track 12.0 -> 96.6 mm, vias 0 -> 2
- net N$45: track 11.9 -> 87.6 mm, vias 0 -> 2
- net TX: track 0.00 -> 72.8 mm
- net RX: track 0.00 -> 71.0 mm
- net VCC: track 63.1 -> 116.7 mm
- net LED_G: track 23.9 -> 75.4 mm, vias 0 -> 2
- net 2.5V: track 1.27 -> 31.3 mm, vias 0 -> 3
- net N$14: track 0.00 -> 28.1 mm, vias 0 -> 1
- net N$13: track 0.05 -> 26.0 mm, vias 0 -> 1
- net N$31: track 0.00 -> 23.5 mm, vias 0 -> 3
- net BLE_TX: track 70.5 -> 51.3 mm, vias 0 -> 2
- net N$5: track 6.98 -> 22.3 mm, vias 0 -> 2
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- added copper zone on layer 1, net 2.5V
- added copper zone on layer 1, net 3.3V
- added copper zone on layer 1, net 5V

Commit message: Update
Parts:
- moved TP6 39.0 mm to (29.5, 31.9)
- moved TP2 20.8 mm to (25.4, 46.4)
- moved C12 4.53 mm to (35.5, 112.8), turned to 180 degrees
- moved D2 2.05 mm to (25.4, 52.5)
- moved R16 1.73 mm to (8.10, 90.1), turned to 270 degrees
- moved C11 1.22 mm to (34.5, 93.9), turned to 90 degrees
- moved C16 1.22 mm to (26.9, 60.1)
- moved C15 1.21 mm to (25.5, 54.8)
- moved C17 0.51 mm to (20.6, 58.6)
- moved F1 0.25 mm to (24.6, 58.3)
Routing:
- net PWR_OUT: track 158.6 -> 139.9 mm, vias 2 -> 6
- net PWR_IN: track 131.3 -> 115.7 mm, vias 2 -> 4
- net N$9: track 96.6 -> 81.4 mm
- net N$45: track 87.6 -> 74.5 mm, vias 2 -> 4
- net GND: track 99.4 -> 109.1 mm
- net N$17: track 18.6 -> 22.9 mm
- net RESET: track 146.3 -> 143.6 mm
- net TX: track 72.8 -> 70.3 mm
- net RX: track 71.0 -> 68.5 mm
- net N$33: track 10.1 -> 8.04 mm
- net LED_G: track 75.4 -> 74.5 mm
- net N$25: track 47.3 -> 46.6 mm
- net N$14: track 28.1 -> 27.4 mm
- net BUT_L: track 41.4 -> 40.7 mm
- net N$28: track 49.4 -> 48.8 mm
- added copper zone on layer 1, net VCC

Commit message: update silkscreen
Parts:
- moved TP1 13.2 mm to (35.1, 14.4)
- moved TP8 2.04 mm to (23.1, 127.8)
- moved LED3 1.02 mm to (19.7, 75.8)
- moved R24 1.02 mm to (24.3, 75.8)
- moved R27 0.76 mm to (10.9, 6.78)
- moved TP4 0.61 mm to (7.54, 122.9)
- moved TP5 0.51 mm to (22.1, 115.3)
- moved TP6 0.51 mm to (30.0, 31.9)
- moved R28 0.51 mm to (13.0, 6.78)
- moved TP9 0.13 mm to (36.9, 127.3)
Routing:
- net N$8: track 5.26 -> 11.2 mm
- net GND: track 109.1 -> 112.7 mm
- net VIN: track 16.4 -> 18.3 mm
- net N$44: track 32.1 -> 31.1 mm
- net LED_G: track 74.5 -> 73.8 mm
Other:
- board text added: "ICSP"
- board text added: "ON/OFF"
- board text added: "RESET"
