File: project/contactless-thermometer.brd (EAGLE design)
At the start: 50 x 150 mm, 94 parts, among them J1 OLED, J2 ICSP, J3 BLE, J4 USB-MINIB-5PIN, Q1 MMBT3904, Q2 MMBT3904, Q3 ZXMP6A17GTA, U1 LT1167CS8#PBF, U2 OPA2705UA, U3 OPA705NA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

Commit message: just wonderful
Parts:
- moved TP8 2.84 mm to (23.9, 127.8)
- moved TP2 1.70 mm to (25.4, 44.7)
- moved C21 0.51 mm to (32.3, 11.6)
- moved R10 0.25 mm to (33.3, 22.5)
- moved R9 0.25 mm to (31.5, 22.5)
- moved C7 0.25 mm to (32.3, 14.1)
- moved TP1 0.25 mm to (35.1, 14.1)
- moved R30 0.18 mm to (33.3, 141.6)
- moved R31 0.13 mm to (33.3, 144.4)
Routing:
- net VR: track 60.4 -> 61.4 mm
- net GND: track 117.0 -> 117.8 mm
- net TX: track 71.6 -> 71.0 mm
- net N$36: track 7.93 -> 7.41 mm

Commit message: update schematics
Parts:
- C2: value 0.1uF -> 0.47uF
- C5: value 0.1uF -> 10nF
- C6: value 0.1uF -> 4.7nF
- U4: value TPS561201 -> TPS562200DDCR
- U5: value ATMEGA328-AU -> ATMEGA328P-AU
Changed lines of the file:
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@@
 <drawing>
 <settings>
-<setting alwaysvectorfont="yes"/>
+<setting alwaysvectorfont="no"/>
 <setting verticaltext="up"/>
 </settings>
@@
 <attribute name="NAME" x="13.462" y="132.715" size="0.6096" layer="25" font="vector" ratio="20" rot="R270" align="bottom-center"/>
 </element>
-<element name="U4" library="SamacSys_Parts" package="SOT95P280X110-6N" value="TPS561201" x="32.258" y="17.9578" smashed="yes" rot="R90" grouprefs="WEBENCH">
+<element name="U4" library="SamacSys_Parts" package="SOT95P280X110-6N" value="TPS562200DDCR" x="32.258" y="17.9578" smashed="yes" rot="R90" grouprefs="WEBENCH">
 <attribute name="DESCRIPTION" value="4.5V to 17V Input, 1A Synchronous Step-Down Voltage Regulator in 6-pin SOT-23" x="105.918" y="58.5978" size="1.778" layer="27" rot="R90" display="off"/>
 <attribute name="HEIGHT" value="1.1mm" x="105.918" y="58.5978" size="1.778" layer="27" rot="R90" display="off"/>
@@
 <attribute name="NAME" x="34.2138" y="17.9578" size="0.6096" layer="25" font="vector" ratio="20" align="center-left"/>
 </element>
-<element name="U5" library="atmel" library_urn="urn:adsk.eagle:library:105" package="TQFP32-08" package3d_urn="urn:adsk.eagle:package:4313/2" value="ATMEGA328-AU" x="22.352" y="106.8578" smashed="yes" rot="R180">
+<element name="U5" library="atmel" library_urn="urn:adsk.eagle:library:105" package="TQFP32-08" package3d_urn="urn:adsk.eagle:package:4313/2" value="ATMEGA328P-AU" x="22.352" y="106.8578" smashed="yes" rot="R180">
 <attribute name="MF" value="" x="3.302" y="150.0378" size="1.778" layer="27" rot="R180" display="off"/>
 <attribute name="MPN" value="ATMEGA8-16AU" x="3.302" y="150.0378" size="1.778" layer="27" rot="R180" display="off"/>
@@
 <attribute name="PROD_ID" value="CAP-00810" x="5.842" y="121.412" size="1.778" layer="27" rot="R270" display="off"/>
 </element>
-<element name="C2" library="SparkFun-Capacitors" package="0603" value="0.1uF" x="14.224" y="120.0658" smashed="yes" rot="R90">
+<element name="C2" library="SparkFun-Capacitors" package="0603" value="0.47uF" x="14.224" y="120.0658" smashed="yes" rot="R90">
 <attribute name="NAME" x="14.224" y="121.92" size="0.6096" layer="25" font="vector" ratio="20" align="bottom-center"/>
 <attribute name="PROD_ID" value="CAP-00810" x="14.224" y="120.0658" size="1.778" layer="27" rot="R90" display="off"/>
 </element>
-<element name="C6" library="SparkFun-Capacitors" package="0603" value="0.1uF" x="33.02" y="120.3198" smashed="yes">
+<element name="C6" library="SparkFun-Capacitors" package="0603" value="4.7nF" x="33.02" y="120.3198" smashed="yes">
 <attribute name="NAME" x="33.02" y="121.158" size="0.6096" layer="25" font="vector" ratio="20" align="bottom-center"/>
 <attribute name="PROD_ID" value="CAP-00810" x="33.02" y="120.3198" size="1.778" layer="27" display="off"/>
 </element>
-<element name="C5" library="SparkFun-Capacitors" package="0603" value="0.1uF" x="26.416" y="121.0818" smashed="yes" rot="R90">
+<element name="C5" library="SparkFun-Capacitors" package="0603" value="10nF" x="26.416" y="121.0818" smashed="yes" rot="R90">
 <attribute name="NAME" x="26.416" y="123.3678" size="0.6096" layer="25" font="vector" ratio="20" rot="R180" align="bottom-center"/>
 <attribute name="PROD_ID" value="CAP-00810" x="26.416" y="121.0818" size="1.778" layer="27" rot="R90" display="off"/>
